File: Flight computer/Hardware/circuit board design v1.1/circuit board design.kicad_pcb (KiCad board)
At the start: 4 copper layers, 30.5 x 82.6 mm, 86 parts, among them J1 Conn_01x05, J2 USB_B_Micro, J3 Screw_Terminal_01x04, J4 Conn_01x02, J5 Conn_01x04, J6 Conn_Coaxial, J7 Conn_Coaxial, U1 LSM9DS1, U11 W25Q64JVSSIM, U14 MAX40200AUK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

Commit message: did some shrinkifying
Not sure if this is the way to go
Parts:
- C11, C14, C15, C16, C17, C20, C21, C23, C24, C25, C3, C34, C4, C6, C7, C77, C86, C88, C89, C91, C93: footprint Capacitor_SMD:C_0603_1608Metric -> Capacitor_SMD:C_0402_1005Metric
- D1, D2: footprint LED_SMD:LED_0603_1608Metric -> LED_SMD:LED_0402_1005Metric
- R1, R12, R13, R15, R16, R25, R26, R28, R29, R3, R4, R5, R6, R8: footprint Resistor_SMD:R_0603_1608Metric -> Capacitor_SMD:C_0402_1005Metric
- moved J7 213.4 mm to (120.0, 275.0)
- moved H1 206.4 mm to (103.8, 267.8), turned to 0 degrees
- moved ANT1 201.5 mm to (108.1, 275.5), turned to 0 degrees
- moved U2 200.6 mm to (115.2, 267.8), turned to 180 degrees
- moved R7 200.3 mm to (107.0, 262.0)
- moved C10 199.9 mm to (107.0, 260.0), turned to 0 degrees
- moved L3 196.3 mm to (107.7, 258.0)
- moved C9 196.2 mm to (109.9, 260.0), turned to 0 degrees
- moved X1 196.0 mm to (113.0, 263.5), turned to 0 degrees
- moved U3 195.1 mm to (110.0, 267.7), turned to 180 degrees
- moved L8 194.5 mm to (96.4, 263.3), turned to 0 degrees
- moved C21 192.9 mm to (96.8, 259.3), turned to 0 degrees
- moved C22 192.9 mm to (92.4, 263.3), turned to 0 degrees
- moved C19 188.8 mm to (107.7, 256.0), turned to 0 degrees
- moved U6 184.3 mm to (117.5, 262.9), turned to 270 degrees
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Routing:
- net GND: track 172.6 -> 0.00 mm, vias 53 -> 0
- net +3V3: track 113.5 -> 0.00 mm, vias 25 -> 0
- net /gps/GPS_SCL: track 72.8 -> 0.00 mm, vias 3 -> 0
- net /gps/GPS_SDA: track 60.8 -> 0.00 mm, vias 2 -> 0
- net /gps/GPS_NRES: track 39.0 -> 0.00 mm, vias 2 -> 0
- net Vdrive: track 38.2 -> 0.00 mm
- net /MCU/MCU_NSEL1: track 36.9 -> 0.00 mm, vias 2 -> 0
- net Net-(C35-Pad1): track 34.7 -> 0.00 mm, vias 2 -> 0
- net /MCU/MCU_PA13: track 34.4 -> 0.00 mm
- net /MCU/MCU_PA12: track 33.6 -> 0.00 mm
- net /gps/GPS_NSAFEBOOT: track 33.6 -> 0.00 mm
- net /MCU/MCU_MISO1: track 32.8 -> 0.00 mm, vias 2 -> 0
- net /MCU/MCU_PB11: track 32.5 -> 0.00 mm, vias 2 -> 0
- net /MCU/MCU_PB10: track 32.2 -> 0.00 mm, vias 2 -> 0
- net /MCU/MCU_SCLK4: track 30.8 -> 0.00 mm, vias 2 -> 0
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- removed copper zone on VCC.Cu, net +3V3
- removed copper zone on B.Cu, net GND
- removed copper zone on F.Cu, net GND
- removed copper zone on GND.Cu, net GND
Other:
- board size 30.5 x 82.6 mm -> 25 x 70 mm
- board text removed: "Board is 4 layer JLCPCB Type JLC7628 1.6mm overall thickness Layer 1 RF and Signal 1oz copper Insulator .2mm 4.6 dielectric constant Layer 2 Ground 1/2 oz copper Insulator 1.065mm 4.6 dielectric constant Layer 3 Power 1/2oz copper Insulator 0.2mm 4.6 dielectric constant Layer 4 Signal 1oz copper Layer 1-2 50 ohm Microstrip width 11.55mil"
- board text removed: "Rocket Flight Computer v1.0 Imperial College Space Society Medad Newman, Richard Ibbotson Sept 2019"
