File: Flight computer/Hardware/circuit board design v1.1/circuit board design.kicad_pcb (KiCad board)
At the start: 4 copper layers, 30.5 x 82.6 mm, 87 parts, among them J1 Conn_01x05, J2 USB_B_Micro, J3 Screw_Terminal_01x04, J4 Conn_01x02, J5 Conn_01x04, J6 Conn_Coaxial, J7 Conn_Coaxial, U1 LSM9DS1, U11 W25Q64JVSSIM, U14 MAX40200AUK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

Commit message: tried to fit in the sma connector. Not really finished
Parts:
- removed G***: LOGO, flight-computer:ICSS_Logo
- J7: footprint Connector_Coaxial:U.FL_Hirose_U.FL-R-SMT-1_Vertical -> Connector_Coaxial:SMA_Molex_73251-1153_EdgeMount_Horizontal
- moved R7 5.51 mm to (107.6, 66.7), turned to 90 degrees
- moved C10 4.86 mm to (101.1, 64.7)
- moved L3 4.86 mm to (101.6, 66.3)
- moved J7 4.57 mm to (108.7, 62.9), turned to 270 degrees
- moved C20 3.02 mm to (112.5, 73.9)
- moved C21 3.02 mm to (114.9, 73.4)
- moved C23 3.02 mm to (103.1, 75.4)
- moved L8 3.02 mm to (103.2, 71.9)
- moved X1 3.02 mm to (114.0, 70.4)
- moved C9 3.02 mm to (108.7, 66.7)
- moved C19 3.02 mm to (103.5, 70.1)
- moved C22 3.02 mm to (103.1, 73.7)
- moved U2 3.02 mm to (107.7, 70.2)
- moved U3 3.02 mm to (107.6, 75.6)
Routing:
- net GND: track 170.7 -> 162.2 mm, vias 53 -> 51
- net Net-(ANT1-Pad1): track 10.7 -> 6.53 mm
- net Net-(J7-Pad1): track 1.50 -> 5.52 mm
- net /MCU/MCU_PB11: track 32.5 -> 29.8 mm
- net Net-(C9-Pad1): track 8.33 -> 7.41 mm
